Commit message: 04081729

File: models/speedbot_v4/speedbot_v4.urdf (robot description, URDF)
Before this commit: robot sbt, 31 links, 30 joints
Joints:
- joint left_elbow_joint: origin xyz=0 0.197 0.0135 rpy=0 0 -1.4 -> xyz=0 0.197 0.0135 rpy=0 0 0
- joint left_shoulder_pitch_joint: origin xyz=0.0080635 0.098693 0.42818 rpy=0 0.3 0 -> xyz=0.0080635 0.098693 0.42818 rpy=0 0 0
- joint left_shoulder_roll_joint: origin xyz=0.0444 0.14081 0.00087012 rpy=-1.4 0 0 -> xyz=0.0444 0.14081 0.00087012 rpy=0 0 0
- joint right_elbow_joint: origin xyz=0 -0.197 0.0135 rpy=0 0 1.4 -> xyz=0 -0.197 0.0135 rpy=0 0 0
- joint right_shoulder_pitch_joint: origin xyz=0.0080635 -0.098693 0.42818 rpy=0 0.3 0 -> xyz=0.0080635 -0.098693 0.42818 rpy=0 0 0
- joint right_shoulder_roll_joint: origin xyz=0.0444 -0.14081 0.00087012 rpy=1.4 0 0 -> xyz=0.0444 -0.14081 0.00087012 rpy=0 0 0

Commit message: 修改urdf，腰部手臂顺序

File: models/speedbot_v4/speedbot_v4.urdf (robot description, URDF)
Before this commit: robot sbt, 31 links, 30 joints
Joints:
- joint left_shoulder_pitch_joint: origin xyz=0.0080635 0.098693 0.42818 rpy=0 0 0 -> xyz=0 0.098693 0.07088 rpy=0 0 0; parent base_link -> upper_body_link
- joint right_shoulder_pitch_joint: origin xyz=0.0080635 -0.098693 0.42818 rpy=0 0 0 -> xyz=0 -0.098693 0.07088 rpy=0 0 0; parent base_link -> upper_body_link

Commit message: "fix 腰部关节"

File: models/speedbot_v4/speedbot_v4.urdf (robot description, URDF)
Before this commit: robot sbt, 31 links, 30 joints
Joints:
- joint waist_yaw_joint: axis 0 0 1 -> (none); limit lower=-3.14 upper=3.14 effort=69 velocity=4.4 -> (none); type revolute -> fixed

Commit message: 对齐 base_link Z 轴与 waist_yaw/IMU 轴线

File: models/speedbot_v4/speedbot_v4.urdf (robot description, URDF)
Before this commit: robot sbt, 31 links, 30 joints
Joints:
- joint left_hip_roll_joint: origin xyz=-0.11644 0.1225 -0.04795 rpy=0 0 0 -> xyz=-0.1245035 0.1225 -0.04795 rpy=0 0 0
- joint right_hip_roll_joint: origin xyz=-0.11644 -0.1225 -0.04795 rpy=0 0 0 -> xyz=-0.1245035 -0.1225 -0.04795 rpy=0 0 0
- joint waist_yaw_joint: origin xyz=0.0080635 0 0.0573 rpy=0 0 0 -> xyz=0 0 0.0573 rpy=0 0 0

File: models/speedbot_v4/speedbot_v4_leg.urdf (robot description, URDF)
Before this commit: robot sbt, 31 links, 30 joints
Joints:
- joint left_hip_roll_joint: origin xyz=-0.11644 0.1225 -0.04795 rpy=0 0 0 -> xyz=-0.1245035 0.1225 -0.04795 rpy=0 0 0
- joint left_shoulder_pitch_joint: origin xyz=0.0080635 0.098693 0.42818 rpy=0 0 0 -> xyz=0 0.098693 0.42818 rpy=0 0 0
- joint right_hip_roll_joint: origin xyz=-0.11644 -0.1225 -0.04795 rpy=0 0 0 -> xyz=-0.1245035 -0.1225 -0.04795 rpy=0 0 0
- joint right_shoulder_pitch_joint: origin xyz=0.0080635 -0.098693 0.42818 rpy=0 0 0 -> xyz=0 -0.098693 0.42818 rpy=0 0 0
- joint waist_yaw_joint: origin xyz=0.0080635 0 0.0573 rpy=0 0 0 -> xyz=0 0 0.0573 rpy=0 0 0
